Commit message: ur robot with working griperrs

File: ur_moveit_config/srdf/ur_macro.srdf.xacro (robot description, xacro)
@@ -5,5 +5,5 @@
     A URDF file must exist for this robot as well, where the joints and the links that are referenced are defined
 -->
-  <xacro:macro name="ur_srdf" params="">
+  <xacro:macro name="ur_srdf" params="tip_link:=tool0 add_gripper_states:=false">
     <!--GROUPS - Representation of a set of joints and links. This can be useful for specifying DOF to plan for, defining arms, end effectors, etc-->
     <!--LINKS - When a link is specified, the parent joint of that link (if it exists) is automatically included-->
@@ -12,5 +12,5 @@
     <!--SUBGROUPS - Groups can also be formed by referencing to already defined group names-->
     <group name="ur_manipulator">
-      <chain base_link="base_link" tip_link="tool0" />
+      <chain base_link="base_link" tip_link="${tip_link}" />
     </group>
     <!--GROUP STATES - Purpose - Define a named state for a particular group, in terms of joint values. This is useful to define states like 'folded arms'-->
@@ -22,4 +22,7 @@
       <joint name="wrist_2_joint" value="0" />
       <joint name="wrist_3_joint" value="0" />
+      <xacro:if value="${add_gripper_states == True or add_gripper_states == 'true'}">
+        <joint name="robotiq_85_left_knuckle_joint" value="0" />
+      </xacro:if>
     </group_state>
     <group_state name="up" group="ur_manipulator">
@@ -30,4 +33,7 @@
       <joint name="wrist_2_joint" value="0" />
       <joint name="wrist_3_joint" value="0" />
+      <xacro:if value="${add_gripper_states == True or add_gripper_states == 'true'}">
+        <joint name="robotiq_85_left_knuckle_joint" value="0" />
+      </xacro:if>
     </group_state>
     <group_state name="test_configuration" group="ur_manipulator">
@@ -38,4 +44,7 @@
       <joint name="wrist_2_joint" value="-1.6" />
       <joint name="wrist_3_joint" value="-0.11" />
+      <xacro:if value="${add_gripper_states == True or add_gripper_states == 'true'}">
+        <joint name="robotiq_85_left_knuckle_joint" value="0" />
+      </xacro:if>
     </group_state>
     <!--END EFFECTOR - Purpose - Represent information about an end effector.-->

Commit message: Multiple robots working without cameras

File: ur_moveit_config/srdf/ur_macro.srdf.xacro (robot description, xacro)
@@ -48,4 +48,16 @@
       </xacro:if>
     </group_state>
+    <!--gripper_test: RViz goal state in deg: pan -54, lift -137, elbow 132, w1 -170, w2 -38, w3 -5-->
+    <group_state name="gripper_test" group="ur_manipulator">
+      <joint name="elbow_joint" value="2.30383" />
+      <joint name="shoulder_lift_joint" value="-2.3911" />
+      <joint name="shoulder_pan_joint" value="-0.94248" />
+      <joint name="wrist_1_joint" value="-2.96706" />
+      <joint name="wrist_2_joint" value="-0.66323" />
+      <joint name="wrist_3_joint" value="-0.08727" />
+      <xacro:if value="${add_gripper_states == True or add_gripper_states == 'true'}">
+        <joint name="robotiq_85_left_knuckle_joint" value="0" />
+      </xacro:if>
+    </group_state>
     <!--END EFFECTOR - Purpose - Represent information about an end effector.-->
     <!--VIRTUAL JOINT - Purpose - this element defines a virtual joint between a robot link and an external frame of reference (considered fixed with respect to the robot)-->

File: ur_moveit_config/srdf/ur_robotiq.srdf.xacro (robot description, xacro)
@@ -4,5 +4,7 @@
   <xacro:include filename="$(find ur_moveit_config)/srdf/ur_macro.srdf.xacro"/>
   <xacro:include filename="$(find ur_moveit_config)/srdf/ur_robotiq_disable_collisions.srdf.xacro"/>
-  <xacro:ur_srdf tip_link="robotiq_85_left_finger_tip_link" add_gripper_states="true"/>
+  <!-- Chain must end at tool0 so trajectories use only the 6 arm joints (scaled_joint_trajectory_controller).
+       The gripper joint is driven by robotiq_gripper_controller (GripperAction), not FollowJointTrajectory. -->
+  <xacro:ur_srdf tip_link="tool0" add_gripper_states="false"/>
   <xacro:ur_robotiq_disable_collisions/>
 </robot>

File: ur_moveit_config/srdf/ur_robotiq_disable_collisions.srdf.xacro (robot description, xacro)
@@ -22,4 +22,7 @@
     <disable_collisions link1="robotiq_85_left_finger_link" link2="robotiq_85_left_finger_tip_link" reason="Adjacent" />
     <disable_collisions link1="robotiq_85_right_finger_link" link2="robotiq_85_right_finger_tip_link" reason="Adjacent" />
+    <!-- Parallel linkage: coarse collision meshes overlap at nominal pose (false self-collision). -->
+    <disable_collisions link1="robotiq_85_left_finger_tip_link" link2="robotiq_85_left_inner_knuckle_link" reason="Adjacent" />
+    <disable_collisions link1="robotiq_85_right_finger_tip_link" link2="robotiq_85_right_inner_knuckle_link" reason="Adjacent" />
     <disable_collisions link1="robotiq_85_left_inner_knuckle_link" link2="robotiq_85_left_finger_link" reason="Never" />
     <disable_collisions link1="robotiq_85_right_inner_knuckle_link" link2="robotiq_85_right_finger_link" reason="Never" />

Commit message: Add Robotiq gripper support and launch configuration updates

File: ur_moveit_config/srdf/ur_macro.srdf.xacro (robot description, xacro)
@@ -5,5 +5,5 @@
     A URDF file must exist for this robot as well, where the joints and the links that are referenced are defined
 -->
-  <xacro:macro name="ur_srdf" params="tip_link:=tool0 add_gripper_states:=false">
+  <xacro:macro name="ur_srdf" params="tip_link:=tool0 add_gripper_states:=false add_gripper_group:=false">
     <!--GROUPS - Representation of a set of joints and links. This can be useful for specifying DOF to plan for, defining arms, end effectors, etc-->
     <!--LINKS - When a link is specified, the parent joint of that link (if it exists) is automatically included-->
@@ -60,4 +60,18 @@
       </xacro:if>
     </group_state>
+    <xacro:if value="${add_gripper_group == True or add_gripper_group == 'true'}">
+      <!--GRIPPER - Robotiq 2F-85. Single actuated joint (the other side mimics it).
+          Sim joint is prismatic: 0.0 = open, 0.043 m = fully closed (see robotiq_2f_85_simple_parallel.urdf.xacro).-->
+      <group name="gripper">
+        <joint name="robotiq_85_left_knuckle_joint" />
+      </group>
+      <group_state name="open" group="gripper">
+        <joint name="robotiq_85_left_knuckle_joint" value="0.0" />
+      </group_state>
+      <group_state name="close" group="gripper">
+        <joint name="robotiq_85_left_knuckle_joint" value="0.043" />
+      </group_state>
+      <end_effector name="gripper_ee" parent_link="${tip_link}" group="gripper" parent_group="ur_manipulator" />
+    </xacro:if>
     <!--END EFFECTOR - Purpose - Represent information about an end effector.-->
     <!--VIRTUAL JOINT - Purpose - this element defines a virtual joint between a robot link and an external frame of reference (considered fixed with respect to the robot)-->

File: ur_moveit_config/srdf/ur_robotiq.srdf.xacro (robot description, xacro)
@@ -6,5 +6,5 @@
   <!-- Chain must end at tool0 so trajectories use only the 6 arm joints (scaled_joint_trajectory_controller).
        The gripper joint is driven by robotiq_gripper_controller (GripperAction), not FollowJointTrajectory. -->
-  <xacro:ur_srdf tip_link="tool0" add_gripper_states="false"/>
+  <xacro:ur_srdf tip_link="tool0" add_gripper_states="false" add_gripper_group="true"/>
   <xacro:ur_robotiq_disable_collisions/>
 </robot>

File: ur_moveit_config/srdf/ur_robotiq_disable_collisions.srdf.xacro (robot description, xacro)
@@ -1,5 +1,6 @@
 <?xml version="1.0" encoding="UTF-8"?>
 <robot xmlns:xacro="http://wiki.ros.org/xacro">
-  <!-- Extra disables for PickNik Robotiq 2F-85 mounted on UR tool0 (sim / hardware). -->
+  <!-- Disable collisions for Robotiq 2F-85 on UR tool0.
+       Matches ur_simulation_gz simplified parallel gripper (two knuckle links only). -->
   <xacro:macro name="ur_robotiq_disable_collisions" params="">
     <disable_collisions link1="tool0" link2="robotiq_coupler_link" reason="Adjacent" />
@@ -16,20 +17,7 @@
     <disable_collisions link1="robotiq_85_base_link" link2="robotiq_85_left_knuckle_link" reason="Adjacent" />
     <disable_collisions link1="robotiq_85_base_link" link2="robotiq_85_right_knuckle_link" reason="Adjacent" />
-    <disable_collisions link1="robotiq_85_base_link" link2="robotiq_85_left_inner_knuckle_link" reason="Adjacent" />
-    <disable_collisions link1="robotiq_85_base_link" link2="robotiq_85_right_inner_knuckle_link" reason="Adjacent" />
-    <disable_collisions link1="robotiq_85_left_knuckle_link" link2="robotiq_85_left_finger_link" reason="Adjacent" />
-    <disable_collisions link1="robotiq_85_right_knuckle_link" link2="robotiq_85_right_finger_link" reason="Adjacent" />
-    <disable_collisions link1="robotiq_85_left_finger_link" link2="robotiq_85_left_finger_tip_link" reason="Adjacent" />
-    <disable_collisions link1="robotiq_85_right_finger_link" link2="robotiq_85_right_finger_tip_link" reason="Adjacent" />
-    <!-- Parallel linkage: coarse collision meshes overlap at nominal pose (false self-collision). -->
-    <disable_collisions link1="robotiq_85_left_finger_tip_link" link2="robotiq_85_left_inner_knuckle_link" reason="Adjacent" />
-    <disable_collisions link1="robotiq_85_right_finger_tip_link" link2="robotiq_85_right_inner_knuckle_link" reason="Adjacent" />
-    <disable_collisions link1="robotiq_85_left_inner_knuckle_link" link2="robotiq_85_left_finger_link" reason="Never" />
-    <disable_collisions link1="robotiq_85_right_inner_knuckle_link" link2="robotiq_85_right_finger_link" reason="Never" />
     <disable_collisions link1="robotiq_85_left_knuckle_link" link2="robotiq_85_right_knuckle_link" reason="Never" />
-    <disable_collisions link1="robotiq_85_left_finger_tip_link" link2="robotiq_85_right_finger_tip_link" reason="Never" />
-    <disable_collisions link1="robotiq_85_left_finger_link" link2="robotiq_85_right_finger_link" reason="Never" />
-    <disable_collisions link1="wrist_3_link" link2="robotiq_85_left_finger_tip_link" reason="Never" />
-    <disable_collisions link1="wrist_3_link" link2="robotiq_85_right_finger_tip_link" reason="Never" />
+    <disable_collisions link1="wrist_3_link" link2="robotiq_85_left_knuckle_link" reason="Never" />
+    <disable_collisions link1="wrist_3_link" link2="robotiq_85_right_knuckle_link" reason="Never" />
   </xacro:macro>
 </robot>
